File: Hardware/ACNodeAdaptor/ACNodeAdaptor.kicad_pcb (KiCad board)
At the start: 2 copper layers, 30 x 40 mm, 8 parts, among them J1 Conn_01x02, J2 Conn_01x04_Male, J3 RJ45, U1 ISL8489EIBZ

Commit message: ACNodeAdaptor: Minor change to silkscreen
The ACNode adaptor is actually assembled with a 3.3V RS422 driver, to
support connection to the ACNode. This board modifies the silkscreen to
reflect this.
Other:
- board text added: "3V3"
- board text added: "ACNode Reader Adaptor V1.1"
- board text removed: "5V"
- board text removed: "ACNode Reader Adaptor V1.0"
